File: mother_board/mother3.brd (EAGLE design)
At the start: 116.8 x 50.8 mm, 35 parts

Commit message: update
Parts:
- added LED1, LED2: (no value), adafruit:LED5MM
- added RL7, RL8: (no value), adafruit:0207/10
- REED1: device SparkFun-Connectors:1X02 -> SparkFun-Connectors:1X04
- REED2: device SparkFun-Connectors:1X03 -> SparkFun-Connectors:1X04
- moved R5 9.91 mm to (55.1, 37.8)
- moved R6 9.65 mm to (58.7, 37.8)
- moved REED2 5.59 mm to (65.5, 2.29), turned to 0 degrees
- moved REED1 5.09 mm to (41.9, 2.29)
- moved J2 1.05 mm to (86.6, 39.1)
Connections:
- removed net NXT/STEP/D10: AMIS-30543.3
- new net N$1: LED1.A, RL7.1
- new net N$2: LED2.A, RL8.1
- net +3V3: now also REED2.2; no longer REED2.1
- net A: now also REED1.4; no longer REED1.2
- net A2: now also RL7.2
- net A3: now also REED2.1
- net B: now also REED2.4; no longer REED2.3
- net D13: now also RL8.2
- net GND: now also LED1.K, LED2.K, REED2.3; no longer REED2.2
- net NEXT/STEP/D10: now also AMIS-30543.3
- net OFF: now also REED1.1
- net ON: now also REED1.2
- net SQW/INT/D6: now also REED1.3; no longer REED1.1
Routing:
- net GND: track 0.00 -> 366.2 mm
- net +3V3: track 0.00 -> 234.8 mm, vias 0 -> 1
- net VDD/5V: track 0.00 -> 186.0 mm, vias 0 -> 3
- net S1_NEG: track 0.00 -> 170.9 mm, vias 0 -> 2
- net A3: track 0.00 -> 140.5 mm, vias 0 -> 2
- net BAT/SWITCH-VIN: track 0.00 -> 140.0 mm, vias 0 -> 1
- net S4_NEG: track 0.00 -> 137.5 mm, vias 0 -> 1
- net MISO: track 0.00 -> 129.1 mm, vias 0 -> 2
- net SCL: track 0.00 -> 118.9 mm
- net S2_NEG: track 0.00 -> 113.5 mm, vias 0 -> 4
- net S3_NEG: track 0.00 -> 111.5 mm, vias 0 -> 3
- net D0: track 0.00 -> 110.9 mm
- net SDA: track 0.00 -> 106.1 mm
- net A5: track 0.00 -> 100.0 mm
- net MOSI: track 0.00 -> 98.2 mm, vias 0 -> 4
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Other:
- board text added: "OFF"
- board text added: "ON"
- board text added: "TINGLY-TENTACLE"
- board text added: "ver 0.1"
- board text removed: "TINGLY-TENTACLE VER 0.1"
