File: mother_board/mother3.sch (EAGLE design)
At the start: 35 parts

Commit message: update
Parts:
- added LED1, LED2: (no value), adafruit:LED5MM
- added RL7, RL8: (no value), adafruit:R-US_0207/10
- REED1: device SparkFun-Connectors:CONN_02 -> SparkFun-Connectors:CONN_04
- REED2: device SparkFun-Connectors:CONN_03 -> SparkFun-Connectors:CONN_04
Connections:
- removed net NXT/STEP/D10: AMIS-30543.3
- new net N$1: LED1.A, RL7.1
- new net N$2: LED2.A, RL8.1
- net +3V3: now also REED2.2; no longer REED2.1
- net A: now also REED1.4; no longer REED1.2
- net A2: now also RL7.2
- net A3: now also REED2.1
- net B: now also REED2.4; no longer REED2.3
- net D13: now also RL8.2
- net GND: now also LED1.C, LED2.C, REED2.3; no longer REED2.2
- net NEXT/STEP/D10: now also AMIS-30543.3
- net OFF: now also REED1.1
- net ON: now also REED1.2
- net SQW/INT/D6: now also REED1.3; no longer REED1.1
Other:
- note added: "LEDS"
- note added: "VOLTAGE MEASURE"
Changed lines of the file:
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@@
 <part name="+3V6" library="supply1" deviceset="+3V3" device=""/>
 <part name="+3V7" library="supply1" deviceset="+3V3" device=""/>
-<part name="REED2" library="SparkFun-Connectors" library_urn="urn:adsk.eagle:library:513" deviceset="CONN_03" device="" package3d_urn="urn:adsk.eagle:package:38063/1"/>
-<part name="REED1" library="SparkFun-Connectors" library_urn="urn:adsk.eagle:library:513" deviceset="CONN_02" device="" package3d_urn="urn:adsk.eagle:package:38039/1"/>
 <part name="+3V8" library="supply1" deviceset="+3V3" device=""/>
 <part name="AMIS-1" library="adafruit" library_urn="urn:adsk.eagle:library:420" deviceset="PINHD-1X12" device="-CB"/>
@@
 <part name="R6" library="adafruit" library_urn="urn:adsk.eagle:library:420" deviceset="R-US_" device="0207/10"/>
 <part name="J3" library="SparkFun-Connectors" library_urn="urn:adsk.eagle:library:513" deviceset="CONN_02" device="" package3d_urn="urn:adsk.eagle:package:38039/1"/>
+<part name="RL7" library="adafruit" library_urn="urn:adsk.eagle:library:420" deviceset="R-US_" device="0207/10"/>
+<part name="LED1" library="adafruit" library_urn="urn:adsk.eagle:library:420" deviceset="LED" device="5MM"/>
+<part name="RL8" library="adafruit" library_urn="urn:adsk.eagle:library:420" deviceset="R-US_" device="0207/10"/>
+<part name="LED2" library="adafruit" library_urn="urn:adsk.eagle:library:420" deviceset="LED" device="5MM"/>
+<part name="REED1" library="SparkFun-Connectors" library_urn="urn:adsk.eagle:library:513" deviceset="CONN_04" device="" package3d_urn="urn:adsk.eagle:package:38085/1"/>
+<part name="REED2" library="SparkFun-Connectors" library_urn="urn:adsk.eagle:library:513" deviceset="CONN_04" device="" package3d_urn="urn:adsk.eagle:package:38085/1"/>
 </parts>
 <sheets>
@@
 <text x="-20.32" y="-7.62" size="2.54" layer="91">I2C PULLUPS</text>
 <text x="116.84" y="73.66" size="2.54" layer="91">DF13 I2C CONNECTORS</text>
+<text x="261.62" y="0" size="2.54" layer="91">VOLTAGE MEASURE</text>
+<text x="294.64" y="40.64" size="2.54" layer="91">LEDS</text>
 </plain>
 <instances>
@@
 <instance part="+3V6" gate="G$1" x="185.42" y="20.32"/>
 <instance part="+3V7" gate="G$1" x="-2.54" y="17.78"/>
-<instance part="REED2" gate="J$1" x="60.96" y="-35.56"/>
-<instance part="REED1" gate="G$1" x="30.48" y="-35.56"/>
 <instance part="+3V8" gate="G$1" x="81.28" y="-35.56"/>
 <instance part="AMIS-1" gate="G$1" x="223.52" y="63.5"/>
@@
 <instance part="R6" gate="G$1" x="292.1" y="-33.02" rot="R90"/>
 <instance part="J3" gate="G$1" x="-35.56" y="53.34"/>
+<instance part="RL7" gate="G$1" x="299.72" y="30.48" rot="R90"/>
+<instance part="LED1" gate="G$1" x="299.72" y="22.86"/>
+<instance part="RL8" gate="G$1" x="317.5" y="30.48" rot="R90"/>
+<instance part="LED2" gate="G$1" x="317.5" y="22.86"/>
+<instance part="REED1" gate="G$1" x="33.02" y="-38.1"/>
+<instance part="REED2" gate="G$1" x="63.5" y="-38.1"/>
 </instances>
 <busses>
@@
 </segment>
 <segment>
-<pinref part="REED2" gate="J$1" pin="2"/>
 <wire x1="68.58" y1="-35.56" x2="71.12" y2="-35.56" width="0.1524" layer="91"/>
 <label x="71.12" y="-35.56" size="1.778" layer="95"/>
+<pinref part="REED2" gate="G$1" pin="3"/>
 </segment>
 <segment>
@@
 <wire x1="292.1" y1="-38.1" x2="292.1" y2="-43.18" width="0.1524" layer="91"/>
 <label x="292.1" y="-43.18" size="1.778" layer="95"/>
+</segment>
+<segment>
+<pinref part="LED1" gate="G$1" pin="C"/>
+<wire x1="299.72" y1="17.78" x2="299.72" y2="12.7" width="0.1524" layer="91"/>
+<label x="299.72" y="12.7" size="1.778" layer="95"/>
+</segment>
+<segment>
+<pinref part="LED2" gate="G$1" pin="C"/>
+<wire x1="317.5" y1="17.78" x2="317.5" y2="12.7" width="0.1524" layer="91"/>
+<label x="317.5" y="12.7" size="1.778" layer="95"/>
 </segment>
 </net>
@@
 <label x="254" y="17.78" size="1.778" layer="95"/>
 </segment>
+<segment>
+<pinref part="REED2" gate="G$1" pin="1"/>
+<wire x1="68.58" y1="-40.64" x2="71.12" y2="-40.64" width="0.1524" layer="91"/>
+<label x="71.12" y="-40.64" size="1.778" layer="95"/>
+</segment>
 </net>
 <net name="A2" class="0">
@@
 <wire x1="251.46" y1="20.32" x2="254" y2="20.32" width="0.1524" layer="91"/>
 <label x="254" y="20.32" size="1.778" layer="95"/>
+</segment>
+<segment>
+<pinref part="RL7" gate="G$1" pin="2"/>
+<wire x1="299.72" y1="35.56" x2="294.64" y2="35.56" width="0.1524" layer="91"/>
+<label x="294.64" y="35.56" size="1.778" layer="95"/>
 </segment>
 </net>
@@
 </segment>
 <segment>
-<pinref part="REED2" gate="J$1" pin="1"/>
 <pinref part="+3V8" gate="G$1" pin="+3V3"/>
 <wire x1="81.28" y1="-38.1" x2="68.58" y2="-38.1" width="0.1524" layer="91"/>
+<pinref part="REED2" gate="G$1" pin="2"/>
 </segment>
 <segment>
@@
 <pinref part="JP3" gate="G$1" pin="4"/>
 </segment>
+<segment>
+<pinref part="RL8" gate="G$1" pin="2"/>
+<wire x1="317.5" y1="35.56" x2="312.42" y2="35.56" width="0.1524" layer="91"/>
+<label x="312.42" y="35.56" size="1.778" layer="95"/>
+<label x="312.42" y="35.56" size="1.778" layer="95"/>
+</segment>
 </net>
 <net name="A0" class="0">
@@
 <pinref part="JP3" gate="G$1" pin="7"/>
 </segment>
+<segment>
+<pinref part="AMIS-30543" gate="G$1" pin="3"/>
+<wire x1="190.5" y1="71.12" x2="182.88" y2="71.12" width="0.1524" layer="91"/>
+<label x="167.64" y="71.12" size="1.778" layer="95"/>
+</segment>
 </net>
 <net name="!RESET" class="0">
@@
 <label x="45.72" y="2.54" size="1.778" layer="95"/>
 </segment>
+<segment>
+<pinref part="REED1" gate="G$1" pin="1"/>
+<wire x1="38.1" y1="-40.64" x2="40.64" y2="-40.64" width="0.1524" layer="91"/>
+<label x="40.64" y="-40.64" size="1.778" layer="95"/>
+</segment>
 </net>
 <net name="ON" class="0">
@@
 <wire x1="43.18" y1="5.08" x2="45.72" y2="5.08" width="0.1524" layer="91"/>
 <label x="45.72" y="5.08" size="1.778" layer="95"/>
+</segment>
+<segment>
+<pinref part="REED1" gate="G$1" pin="2"/>
+<wire x1="38.1" y1="-38.1" x2="40.64" y2="-38.1" width="0.1524" layer="91"/>
+<label x="40.64" y="-38.1" size="1.778" layer="95"/>
 </segment>
 </net>
@@
 </segment>
 <segment>
-<pinref part="REED2" gate="J$1" pin="3"/>
 <wire x1="68.58" y1="-33.02" x2="71.12" y2="-33.02" width="0.1524" layer="91"/>
 <label x="71.12" y="-33.02" size="1.778" layer="95"/>
+<pinref part="REED2" gate="G$1" pin="4"/>
 </segment>
 </net>
@@
 <wire x1="38.1" y1="-33.02" x2="40.64" y2="-33.02" width="0.1524" layer="91"/>
 <label x="40.64" y="-33.02" size="1.778" layer="95"/>
-<pinref part="REED1" gate="G$1" pin="2"/>
-</segment>
-</net>
-<net name="NXT/STEP/D10" class="0">
-<segment>
-<pinref part="AMIS-30543" gate="G$1" pin="3"/>
-<wire x1="190.5" y1="71.12" x2="182.88" y2="71.12" width="0.1524" layer="91"/>
-<label x="167.64" y="71.12" size="1.778" layer="95"/>
+<pinref part="REED1" gate="G$1" pin="4"/>
 </segment>
 </net>
@@
 <wire x1="38.1" y1="-35.56" x2="40.64" y2="-35.56" width="0.1524" layer="91"/>
 <label x="40.64" y="-35.56" size="1.778" layer="95"/>
-<pinref part="REED1" gate="G$1" pin="1"/>
+<pinref part="REED1" gate="G$1" pin="3"/>
 </segment>
 <segment>
@@
 </segment>
 </net>
+<net name="N$1" class="0">
+<segment>
+<pinref part="RL7" gate="G$1" pin="1"/>
+<pinref part="LED1" gate="G$1" pin="A"/>
+</segment>
+</net>
+<net name="N$2" class="0">
+<segment>
+<pinref part="RL8" gate="G$1" pin="1"/>
+<pinref part="LED2" gate="G$1" pin="A"/>
+</segment>
+</net>
